Commit message: feat: make the bridged sensors present the interface hardware will
Every sensor in the model stamped its messages with Gazebo's own scoped name,
because none of them set gz_frame_id. Those frames are not in the tree
robot_state_publisher serves, so RViz silently drew nothing and a real driver
would have published different names. The lidar, rangefinder and camera now
carry front_lidar_link, rangefinder_link and camera_optical_frame.

The bridged IMU was the sensor ArduPilot reads, which the model deliberately
rolls 180 degrees into aircraft convention, so it reported -9.81 on z where
REP 103 and AP_DDS both give +9.81. Every ROS consumer would have found its y
and z inverted on real hardware. The model carries a second, unrotated imu_ros
for the bridge now.

/openipc_cinewhoop/range/down carried a LaserScan while spec/04_ros_rozhrani.md
has always specified Range, which is what the MTF-02P driver publishes. The
bridge ends at down_raw and range_adapter owns the logical name. The simulated
sensor is a narrow fan rather than one ray, because a time-of-flight sensor
returns the nearest surface in its cone and one ray left angle_increment NaN.

Both downward sensor frames are pitched 90 degrees in the URDF to match the SDF;
level frames would have put the floor measurement in front of the drone.

The same two model files also carry the corrected wheelbase, which cannot be
split out of them: 126 mm was an assumption and GEPRC publish 128 mm, so the
motor coordinates move from 0.04455 m to 0.04525 m.

check_sensor_interface.sh asserts the shape of the data rather than the names on
the graph: message types against the spec, every frame_id transformable into
base_link, the declared rangefinder cone against the fan actually cast, and
gravity reading +9.81 on the IMU's z.

Co-Authored-By: Claude Opus 5 <noreply@anthropic.com>
Claude-Session: https://claude.ai/code/session_01CEsLBAvyJXgmTJE1gBdUuK

File: ros_ws/src/openipc_cinewhoop_description/urdf/openipc_cinewhoop.urdf.xacro (robot description, xacro)
@@ -1,5 +1,8 @@
 <?xml version="1.0"?>
 <robot xmlns:xacro="http://www.ros.org/wiki/xacro" name="openipc_cinewhoop">
-  <xacro:property name="arm" value="0.04455"/>
+  <!-- Half the 128 mm wheelbase GEPRC publish for the CineLog30 V3, divided by
+       sqrt(2) for the quad X diagonal. The spec carried 126 mm, which was the
+       original assumption rather than the frame's real figure. -->
+  <xacro:property name="arm" value="0.04525"/>
   <xacro:property name="prop_r" value="0.0381"/>
   <material name="carbon"><color rgba="0.04 0.045 0.05 1.0"/></material>
@@ -21,5 +24,5 @@
     </inertial>
   </link>
-  <xacro:macro name="fixed_box_link" params="name xyz size material">
+  <xacro:macro name="fixed_box_link" params="name xyz size material rpy:='0 0 0'">
     <link name="${name}">
       <visual>
@@ -32,5 +35,5 @@
       <parent link="base_link"/>
       <child link="${name}"/>
-      <origin xyz="${xyz}" rpy="0 0 0"/>
+      <origin xyz="${xyz}" rpy="${rpy}"/>
     </joint>
   </xacro:macro>
@@ -62,6 +65,10 @@
   </joint>
   <xacro:fixed_box_link name="imu_link" xyz="0 0 0.018" size="0.018 0.018 0.006" material="sensor"/>
-  <xacro:fixed_box_link name="optical_flow_link" xyz="0 0 -0.016" size="0.018 0.018 0.006" material="sensor"/>
-  <xacro:fixed_box_link name="rangefinder_link" xyz="0.020 0 -0.016" size="0.014 0.014 0.008" material="sensor"/>
+  <!-- Both downward sensors measure along +X of their own frame, so the frames
+       are pitched 90 degrees to point at the floor. The simulated sensor link
+       carries the same rotation; a frame that disagrees with the beam would
+       place the measurement in front of the drone instead of below it. -->
+  <xacro:fixed_box_link name="optical_flow_link" xyz="0 0 -0.016" rpy="0 ${pi/2} 0" size="0.018 0.018 0.006" material="sensor"/>
+  <xacro:fixed_box_link name="rangefinder_link" xyz="0.020 0 -0.016" rpy="0 ${pi/2} 0" size="0.014 0.014 0.008" material="sensor"/>
   <xacro:fixed_box_link name="front_lidar_link" xyz="0.073 0 0.002" size="0.018 0.030 0.014" material="sensor"/>
   <xacro:motor name="motor_1" x="${arm}" y="-${arm}"/>

Commit message: feat: fly the mass the bill of materials actually says
The model flew on 0.240 kg, which was the figure the requirement asked for
rather than one anything was weighed against. The bill of materials with the
LD06 says 0.306 kg, so that is what it flies on now, and the lidar's 42 g sits
on front_lidar_link rather than in base_link because Gazebo composes the body
inertia from where the links are and the whole point is that this mass hangs on
a mast.

That is not a number change. 42 g at 46 mm forward and 50 mm up adds about
1.9e-4 to pitch inertia, as much again as the entire airframe had before, taking
roll inertia from roughly 0.00028 to 0.00045. Hover throttle moved from 0.41 to
0.46 and thrust to weight from 5.9 to 4.6. The tuning stopped being valid with
it: at 0.027 the guided takeoff's worst tilt went from 6.5 to 24.0 degrees,
against the check's 25 degree limit.

So the sweep ran again, which is what it exists for. At 0.306 kg the onset is
between 0.065 and 0.08 - ringing holds at 3 through 0.065, reaches 11 at 0.07,
and at 0.08 the loop is gone with 146 sign changes and 62 per cent overshoot.
ATC_RAT_RLL_P is 0.040, just under six tenths of the onset, the same margin the
previous tuning used. Worst tilt came back to 15.6 degrees, which is not the 6.5
of the lighter airframe and should not be: it carries a lidar on a stick now.

Thrust stand, guided takeoff, forward flight and baseline CI all pass.

Co-Authored-By: Claude Opus 5 <noreply@anthropic.com>
Claude-Session: https://claude.ai/code/session_01CEsLBAvyJXgmTJE1gBdUuK

File: ros_ws/src/openipc_cinewhoop_description/urdf/openipc_cinewhoop.urdf.xacro (robot description, xacro)
@@ -20,6 +20,10 @@
     </collision>
     <inertial>
-      <mass value="0.240"/>
-      <inertia ixx="0.00022" ixy="0" ixz="0" iyy="0.00022" iyz="0" izz="0.00038"/>
+      <!-- The URDF lumps everything here because it only has to look right;
+           the SDF spreads the same 0.306 kg over the links physics acts on.
+           Only the totals are comparable, and check_model_consistency.py
+           compares them. -->
+      <mass value="0.306"/>
+      <inertia ixx="0.00047" ixy="0" ixz="0" iyy="0.00047" iyz="0" izz="0.00048"/>
     </inertial>
   </link>
