Commit message: feat: align the model with what the shopping list actually buys
The uncommitted work from 2026-09-14, landed as one commit because it is one
piece of work: publishing the parts lists found that the simulation and the
bill of materials had drifted apart, and everything here follows from closing
that gap.

models_pavo20/ was built from the airframe study, which chose LAVA 1104 5500KV,
an iFlight Beast H7 and a 750 mAh pack at 0.2216 kg. The costing found the LAVA
is not sold in this country at all, so the list buys Flashhobby A1204 5200KV, a
MicoAir H743 and an 850 mAh pack, and the machine is 0.22934 kg. The model now
follows the list rather than the study: maxRotVelocity 5950 -> 5580, per-link
masses off the itemised budget, MOT_THST_HOVER 0.49 -> 0.53.

That cost an earlier claim. Roll authority is 583 rad/s^2 against the CineLog's
689, a ratio of 0.85 where the LAVA model gave 0.99, so the rate gains no longer
transfer by argument. sweep_rate_gains.sh could not test it - the base parameter
file and the model directory were both hardcoded - so it now takes
OPENIPC_AIRFRAME and writes into logs/rate_sweep/<airframe>-<stamp>/. Measured:
0.065 clean, 0.080 gone, the same bracket as the CineLog, so 0.040 stays and is
now measured rather than argued.

Documents: 08_kalkulace_dopravy.md prices import against domestic per line,
09_kudy_do_ros.md writes out the four paths by which a scan could reach ROS on
real hardware, 12_reserse_motoru.md is the motor search for 4x M2 at 9 mm, and
scripts/nakup_calc.py is the basket calculator the published pages use. The
frame's name is corrected throughout to Pavo20 Pro, not Pro II.

Committed as it stood, to land the branch on main. Waiting, an empty file from
2026-09-12, is left untracked.

Co-Authored-By: Claude Opus 5 <noreply@anthropic.com>

File: ros_ws/src/openipc_cinewhoop_description/urdf/openipc_pavo20.urdf.xacro (robot description, xacro)
@@ -26,9 +26,10 @@
     <inertial>
       <!-- The URDF lumps everything here because it only has to look right;
-           the SDF spreads the same 0.2216 kg over the links physics acts on.
+           the SDF spreads the same 0.22934 kg over the links physics acts on.
            Only the totals are comparable, and check_model_consistency.py
-           compares them. -->
-      <mass value="0.2216"/>
-      <inertia ixx="0.00022" ixy="0" ixz="0" iyy="0.00022" iyz="0" izz="0.00016"/>
+           compares them. The figure is the bill of materials' final machine in
+           spec/realna_stavba_dronu/11_kusovnik_pavo20.md, lidar included. -->
+      <mass value="0.22934"/>
+      <inertia ixx="0.000225" ixy="0" ixz="0" iyy="0.000225" iyz="0" izz="0.000314"/>
     </inertial>
   </link>
