File: dps/aio/aio.kicad_pcb (KiCad board)
At the start: 8 copper layers, 35 x 35 mm, 343 parts, among them J15 5V, J16 5V, J17 5V, J18 5V, J20 5V, J21 5V, J23 5V, J24 5V, J25 5V, J26 5V, J27 5V, J28 5V, J29 5V, J30 5V, J31 5V, J32 5V, J33 5V, J34 5V, J35 5V, J37 5V, J38 5V, J39 5V, J40 5V, J41 5V, J42 5V, J43 5V, J44 5V, J45 5V, J48 5V, J49 5V, J50 5V, J51 5V, J52 5V, J53 5V, J54 5V, J55 5V, Q1 AP1606, Q10 DOY180N03T, Q11 DOY180N03T, Q12 DOY180N03T, Q13 DOY180N03T, Q14 DOY180N03T, Q15 DOY180N03T, Q16 DOY180N03T, Q17 DOY180N03T, Q18 DOY180N03T, Q19 DOY180N03T, Q2 AP1606, Q20 DOY180N03T, Q21 DOY180N03T, Q22 DOY180N03T, Q23 DOY180N03T, Q24 DOY180N03T, Q25 DOY180N03T, Q26 DOY180N03T, Q3 DOY180N03T, Q4 DOY180N03T, Q5 DOY180N03T, Q6 DOY180N03T, Q7 DOY180N03T, Q8 DOY180N03T, Q9 DOY180N03T, U1 TS2306A 240GF MSM 9_C2976675, U10 COS8051SOT, U11 TLV7031DPWR, U12 SM06B-SRSS-TB(LF)(SN), U13 AT32F421G8U7, U14 NSG2065Q, U15 AT32F421G8U7, U16 NSG2065Q, U17 AT32F421G8U7, U18 NSG2065Q, U19 AT32F421G8U7, U2 RP2354A, U20 NSG2065Q, U21 SX1281IMLTRT, U22 ESP32-C3, U24 AIO_outline, U25 INA186A3IDCKR, U26 BMP580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

Commit message: feat: update the AIO board from the schematic, and give the microSD slot its DAT1/DAT2 pads
- gen/aktualizuj_desku.sh does what F8 does, without the GUI: matches
  footprints by UUID path, removes the 145 of the dropped OpenAIO sheets,
  adds the 93 new ones off the board, sets pad nets, keeps the copper of the
  10 nets that only changed name (MOTOR1-4, CURR, the IMU bus) and removes the
  845 items of the 70 nets left on nothing.
- OpenAIO's TF-021B-H265 footprint had no pads 1 (DAT2) and 8 (DAT1): it reads
  the card over SPI. We use 4-bit SDMMC; the part has all 8 contacts, added at
  EasyEDA's positions, into the gaps the silkscreen had left for them.
- DRC with parity: 238 unconnected (new parts), 44 dangling tracks where the
  RP2354 was, the rest are OpenAIO's warnings at the same places.

Co-Authored-By: Claude Opus 5.5 <noreply@anthropic.com>
Parts:
- removed AE2: 2450AT18A100E, lib:ANT-SMD_L3.2-W1.6
- removed C1, C107, C108, C11, C12, C13, C14, C2, C32, C34, C35, C36, C5, C6, C7, C8, C9: 100n, lib:C_0201_0603Metric
- removed C10, C4: 20p, lib:C_0201_0603Metric
- removed C15, C16, C17, C3: 4.7uF, lib:C_0402_1005Metric
- removed C31: 470p, lib:C_0201_0603Metric
- removed C33: 1uF, lib:C_0402_1005Metric
- removed C65, C66, C70, C71, C76, C78, C79: 100nF, lib:C_0201_0603Metric
- removed C67, C73, C80: 10nF, lib:C_0201_0603Metric
- removed C68: 470nF, lib:C_0201_0603Metric
- removed C69: 1nF, lib:C_0201_0603Metric
- removed C72, C74: 15pF, lib:C_0201_0603Metric
- removed C75, C82, C88: 10uF, lib:C_0402_1005Metric
- removed C77, C81, C83, C84, C85, C86: 1uF, lib:C_0201_0603Metric
- removed C87, C89: 1.2pF, lib:C_0201_0603Metric
- removed Card1: TF-021B-H265, lib:TF-SMD_TF-021B-H265
- removed D1: LED_1_Blue, lib:LED_0402_1005Metric
- removed D8: SDM02U30LP3-7B, lib:X3-DFN0603-2_L0.6-W0.3-RD
- removed D9: XL-1010RGBC-WS2812B, lib:LED-SMD_4P-L1.0-W1.0-TL_XL-1010RGBC-WS2812B
- removed FL1: 2450FM07D0034T, lib:FILTER-SMD_4P-L1.0-W0.5-L
- removed J15, J16, J17, J18, J20, J21, J23, J24, J25, J26, J27, J28, J29, J30, J31, J32, J33, J34, J35, J37, J38, J39, J40, J41, J42, J43, J44, J45, J48, J49, J50, J51, J52, J53, J54, J55: 5V, lib:small_pad
- removed JP1: U.FL-R-SMT-1(80), lib:RF-SMD_FRF05002-JSS103M
- removed JP2: ELRS OFF, lib:SolderJumper-2_P0.65mm_Tiny_Open
- removed L1: AOTA-B201610S3R3-101-T, lib:IND-SMD_L2.0-W1.6_AOTA-B201610S3R3-101-T
- removed L4: 15uH, lib:L_0805_2012Metric
- removed L5: 24nH, lib:L_0201_0603Metric
- removed L6: 2.0nH, lib:L_0201_0603Metric
- removed L7: 2.5nH, lib:L_0201_0603Metric
- removed OSC1: OW7EL89CENUNFAYLC-52M, lib:OSC-SMD_4P-L2.0-W1.6-BL_TXC_7Z
- removed Q1, Q2: AP1606, lib:DFN-3L_L1.0-W0.6-P0.65-BR
- removed R1, R13: 100k, lib:R_0201_0603Metric
- removed R10, R8, R9: 30R, lib:R_0201_0603Metric
- removed R11, R12, R3, R4: 5.1k, lib:R_0201_0603Metric
- removed R111, R112, R113, R114, R2, R34, R7: 10k, lib:R_0201_0603Metric
- removed R115, R5, R6: 1k, lib:R_0201_0603Metric
- removed R14: 2.4k, lib:R_0201_0603Metric
- removed R15, R16, R26, R33: 75R, lib:R_0201_0603Metric
- removed R27: 3.9k, lib:R_0201_0603Metric
- removed R28: 12k, lib:R_0201_0603Metric
- removed R29: 1.4k, lib:R_0201_0603Metric
- removed R30: 680R, lib:R_0201_0603Metric
- removed R31, R32: 510R, lib:R_0201_0603Metric
- removed TP9: BOOT, lib:SolderPad_1.2x2.0mm
- removed U1: TS2306A 240GF MSM 9_C2976675, lib:SW-SMD_4P-L3.0-W2.0-P0.85-LS3.5
- removed U10: COS8051SOT, lib:SOT-23-5_L3.0-W1.7-P0.95-LS2.8-BR
- removed U11: TLV7031DPWR, lib:X2SON-4_L0.8-W0.8-P0.48-TL-A
- removed U12: SM06B-SRSS-TB(LF)(SN), lib:CONN-SMD_SM06B-SRSS-TB-LF-SN
- removed U2: RP2354A, lib:QFN-60_L7.0-W7.0-P0.40-TL-EP3.4
- removed U21: SX1281IMLTRT, lib:QFN-24_L4.0-W4.0-P0.50-TL-EP2.6
- removed U22: ESP32-C3, lib:QFN-32-1EP_5x5mm_P0.5mm_EP3.7x3.7mm
- removed U26: BMP580, lib:LGA-10_L2.0-W2.0-P0.50-TL_BMP580
- removed U9: SN74LVC1G3157DTBR, lib:X2SON-6_L1.0-W0.8-BL
- removed USB1: TYPE-C 16P QTWT, lib:USB-TYPE-C-SMD_TYPE-C-16P-QTWT
- removed X1: XTM25012000JT00351001, lib:CRYSTAL-SMD_4P-L2.5-W2.0-BL-A
- removed X2: CJ17-400001010B20, lib:CRYSTAL-SMD_4P-L1.6-W1.2-BL
- added C201: 4.7uF 50v, lib:C_0805_2012Metric, F.Cu at (101.7, 52.6)
- added C202: 100n, lib:C_0201_0603Metric, F.Cu at (105.7, 51.9)
- added C203: 22uF, lib:C_0603_1608Metric, F.Cu at (109.4, 52.3)
- added C204: 100n, lib:C_0201_0603Metric, F.Cu at (113.1, 51.9)
- added C301: 100n, lib:C_0201_0603Metric, F.Cu at (100.7, 40.4)
- added C302: 100n, lib:C_0201_0603Metric, F.Cu at (103.7, 40.4)
- added C303: 100n, lib:C_0201_0603Metric, F.Cu at (106.6, 40.4)
- added C304: 4.7uF, lib:C_0402_1005Metric, F.Cu at (109.8, 40.5)
- added C305: 4.7uF, lib:C_0402_1005Metric, F.Cu at (113.2, 40.5)
- added C306: 2.2uF, lib:C_0402_1005Metric, F.Cu at (116.5, 40.5)
- added C307: 2.2uF, lib:C_0402_1005Metric, F.Cu at (119.9, 40.5)
- added C308: 100n, lib:C_0201_0603Metric, F.Cu at (123.1, 40.4)
- added C309: 1uF, lib:C_0402_1005Metric, F.Cu at (126.2, 40.5)
- added C310: 100n, lib:C_0201_0603Metric, F.Cu at (129.4, 40.4)
- added C311: 1uF, lib:C_0402_1005Metric, F.Cu at (132.5, 40.5)
- added C312: 100n, lib:C_0201_0603Metric, F.Cu at (135.7, 40.4)
- added C313: 100n, lib:C_0201_0603Metric, F.Cu at (138.6, 40.4)
- added C314: 100n, lib:C_0201_0603Metric, F.Cu at (141.6, 40.4)
- added C317: 100n, lib:C_0201_0603Metric, F.Cu at (144.5, 40.4)
- added C318: 100n, lib:C_0201_0603Metric, F.Cu at (147.5, 40.4)
- added C319: 100n, lib:C_0201_0603Metric, F.Cu at (150.4, 40.4)
- added C320: 100n, lib:C_0201_0603Metric, F.Cu at (153.4, 40.4)
- added C321: 4.7uF, lib:C_0402_1005Metric, F.Cu at (156.6, 40.5)
- added C322: 15pF C0G, lib:C_0402_1005Metric, F.Cu at (159.9, 40.5)
- added C323: 15pF C0G, lib:C_0402_1005Metric, F.Cu at (163.3, 40.5)
- added D301: XL-1005SURC, lib:LED_0402_1005Metric, F.Cu at (166.9, 40.5)
- added D302: XL-1005UGC, lib:LED_0402_1005Metric, F.Cu at (170.6, 40.5)
- added D303: XL-1005UBC, lib:LED_0402_1005Metric, F.Cu at (174.2, 40.5)
- added D304: 1N4148WS, Diode_SMD:D_SOD-323, F.Cu at (178.3, 41.0)
- added J201: HD VTX, Connector_JST:JST_SH_SM06B-SRSS-TB_1x06-1MP_P1.00mm_Horizontal, F.Cu at (120.3, 54.9)
- added J202: LD06, Connector_JST:JST_ZH_S4B-ZR-SM4A-TF_1x04-1MP_P1.50mm_Horizontal, F.Cu at (132.0, 55.1)
- added J301: TYPE-C 16P QTWT, lib:USB-TYPE-C-SMD_TYPE-C-16P-QTWT, F.Cu at (187.4, 42.9)
- added J302: TF-021B-H265, lib:TF-SMD_TF-021B-H265, F.Cu at (200.8, 43.2)
- added J303: GPS WS-M181, Connector_JST:JST_SH_SM06B-SRSS-TB_1x06-1MP_P1.00mm_Horizontal, F.Cu at (213.4, 43.3)
- added J304: MTF-02P, Connector_JST:JST_SH_SM04B-SRSS-TB_1x04-1MP_P1.00mm_Horizontal, F.Cu at (223.8, 43.3)
- added JP201: VTX vždy zapnutý, Jumper:SolderJumper-2_P1.3mm_Open_Pad1.0x1.5mm, F.Cu at (140.4, 52.8)
- added JP202: SBUS z DJI, Jumper:SolderJumper-2_P1.3mm_Open_Pad1.0x1.5mm, F.Cu at (145.3, 52.8)
- added L201: XRTC303020D4R7MBCA, lib:IND-SMD_L3.0-W3.0_AFE303020S, F.Cu at (150.1, 53.4)
- added Q301: AO3400A, Package_TO_SOT_SMD:SOT-23, F.Cu at (231.1, 41.7)
- added R201: 100k, lib:R_0201_0603Metric, F.Cu at (153.9, 51.9)
- added R202: 6.49k, lib:R_0201_0603Metric, F.Cu at (156.9, 51.9)
- added R203: 1k, lib:R_0201_0603Metric, F.Cu at (159.8, 51.9)
- added R204: 100k, lib:R_0201_0603Metric, F.Cu at (162.8, 51.9)
- added R205: 20m 1%, Resistor_SMD:R_0805_2012Metric, F.Cu at (166.7, 52.5)
- added R206: 0R, lib:R_0201_0603Metric, F.Cu at (170.6, 51.9)
- added R301: 10k, lib:R_0201_0603Metric, F.Cu at (235.3, 40.4)
- added R302: 10k, lib:R_0201_0603Metric, F.Cu at (238.3, 40.4)
- added R303: 100k, lib:R_0201_0603Metric, F.Cu at (241.2, 40.4)
- added R304: 10k, lib:R_0201_0603Metric, F.Cu at (244.2, 40.4)
- added R305: 2.2k, lib:R_0201_0603Metric, F.Cu at (247.1, 40.4)
- added R306: 2.2k, lib:R_0201_0603Metric, F.Cu at (250.1, 40.4)
- added R307: 5.1k, lib:R_0201_0603Metric, F.Cu at (253.0, 40.4)
- added R308: 5.1k, lib:R_0201_0603Metric, F.Cu at (256.0, 40.4)
- added R309: 47k, lib:R_0201_0603Metric, F.Cu at (258.9, 40.4)
- added R310: 47k, lib:R_0201_0603Metric, F.Cu at (261.9, 40.4)
- added R311: 47k, lib:R_0201_0603Metric, F.Cu at (264.8, 40.4)
- added R312: 47k, lib:R_0201_0603Metric, F.Cu at (267.8, 40.4)
- added R313: 47k, lib:R_0201_0603Metric, F.Cu at (270.7, 40.4)
- added R314: 4.7k, lib:R_0201_0603Metric, F.Cu at (273.7, 40.4)
- added R315: 4.7k, lib:R_0201_0603Metric, F.Cu at (276.6, 40.4)
- added R316: 330R, lib:R_0201_0603Metric, F.Cu at (279.6, 40.4)
- added R317: 150R, lib:R_0201_0603Metric, F.Cu at (282.5, 40.4)
- added R318: 75R, lib:R_0201_0603Metric, F.Cu at (285.5, 40.4)
- added R319: 100k, lib:R_0201_0603Metric, F.Cu at (288.4, 40.4)
- added TP301: BOOT0, lib:TestPoint_Pad_D1.0mm, F.Cu at (291.7, 41.0)
- added TP302: +3.3V, lib:TestPoint_Pad_D1.0mm, F.Cu at (295.2, 41.0)
- added TP303: SWDIO, lib:TestPoint_Pad_D1.0mm, F.Cu at (298.8, 41.0)
- added TP304: SWCLK, lib:TestPoint_Pad_D1.0mm, F.Cu at (302.3, 41.0)
- added TP305: NRST, lib:TestPoint_Pad_D1.0mm, F.Cu at (305.9, 41.0)
- added TP306: GND, lib:TestPoint_Pad_D1.0mm, F.Cu at (309.4, 41.0)
- added TP307: XR1 5V, lib:TestPoint_Pad_D1.0mm, F.Cu at (313.0, 41.0)
- added TP308: XR1 GND, lib:TestPoint_Pad_D1.0mm, F.Cu at (316.5, 41.0)
- added TP309: XR1 TX, lib:TestPoint_Pad_D1.0mm, F.Cu at (320.1, 41.0)
- added TP310: XR1 RX, lib:TestPoint_Pad_D1.0mm, F.Cu at (323.6, 41.0)
- added TP311: UART1 TX, lib:TestPoint_Pad_D1.0mm, F.Cu at (327.2, 41.0)
- added TP312: UART1 RX, lib:TestPoint_Pad_D1.0mm, F.Cu at (330.7, 41.0)
- added TP313: UART8 TX, lib:TestPoint_Pad_D1.0mm, F.Cu at (334.3, 41.0)
- added TP314: UART8 RX, lib:TestPoint_Pad_D1.0mm, F.Cu at (337.8, 41.0)
- added TP315: PWM5, lib:TestPoint_Pad_D1.0mm, F.Cu at (341.4, 41.0)
- added TP316: PWM7, lib:TestPoint_Pad_D1.0mm, F.Cu at (344.9, 41.0)
- added TP317: PWM9, lib:TestPoint_Pad_D1.0mm, F.Cu at (348.5, 41.0)
- added TP318: PWM10, lib:TestPoint_Pad_D1.0mm, F.Cu at (352.0, 41.0)
- added TP319: PWM11, lib:TestPoint_Pad_D1.0mm, F.Cu at (355.6, 41.0)
- added TP320: 5V, lib:TestPoint_Pad_D1.0mm, F.Cu at (359.1, 41.0)
- added TP321: GND, lib:TestPoint_Pad_D1.0mm, F.Cu at (362.7, 41.0)
- added TP322: BZ+, lib:TestPoint_Pad_D1.0mm, F.Cu at (366.2, 41.0)
- added TP323: BZ-, lib:TestPoint_Pad_D1.0mm, F.Cu at (369.8, 41.0)
- added U201: LMR51430YFDDCR, lib:SOT-23-6_L2.9-W1.6-P0.95-LS2.9-BL, F.Cu at (174.8, 53.2)
- added U202: INA226AIDGSR, Package_SO:TSSOP-10_3x3mm_P0.5mm, F.Cu at (181.1, 53.4)
- added U301: STM32H743VIH6, Package_BGA:TFBGA-100_8x8mm_Layout10x10_P0.8mm, F.Cu at (377.3, 45.0)
- added U302: SPL06-001 / DPS310, Package_LGA:Bosch_LGA-8_2x2.5mm_P0.65mm_ClockwisePinNumbering, F.Cu at (385.6, 41.5)
- added U303: BMI088, Package_LGA:Bosch_LGA-16_4.5x3mm_P0.5mm_LayoutBorder7x1y_ClockwisePinNumbering, F.Cu at (391.4, 41.9)
- added Y301: 8MHz 12pF X32258MOB4SI, Crystal:Crystal_SMD_3225-4Pin_3.2x2.5mm, F.Cu at (397.7, 41.8)
Connections:
- net /IMU/CS renamed /IMU_CS
- R39 pad 1: MOTOR1 -> /MOTOR1
- R58 pad 1: MOTOR2 -> /MOTOR2
- R77 pad 1: MOTOR3 -> /MOTOR3
- R96 pad 1: MOTOR4 -> /MOTOR4
- U25 pad 6: CURR -> /ESC_CURRENT
- U8 pad 1: /IMU/SPI1.MISO -> /IMU_SPI.MISO
- U8 pad 13: /IMU/SPI1.SCK -> /IMU_SPI.SCK
- U8 pad 14: /IMU/SPI1.MOSI -> /IMU_SPI.MOSI
- U8 pad 4: /IMU/GYRO_INT -> /IMU_INT
Routing:
- net LED_STRIP: track 121.6 -> 0.00 mm, vias 10 -> 0
- net UART1_RX: track 28.3 -> 0.00 mm, vias 8 -> 0
- net USB_D+: track 27.7 -> 0.00 mm, vias 5 -> 0
- net USB_D-: track 27.6 -> 0.00 mm, vias 7 -> 0
- net UART1_TX: track 24.4 -> 0.00 mm, vias 5 -> 0
- net BUZZER-: track 24.0 -> 0.00 mm, vias 4 -> 0
- net CURR: track 21.5 -> 0.00 mm, vias 4 -> 0
- net /ESC_CURRENT: track 0.00 -> 21.5 mm, vias 0 -> 4
- net /RX/CHIP_EN: track 20.1 -> 0.00 mm, vias 6 -> 0
- net /RX/NSS: track 18.9 -> 0.00 mm, vias 4 -> 0
- net /RX/MOSI: track 18.5 -> 0.00 mm, vias 4 -> 0
- net /Pads/I2C0.SDA: track 18.1 -> 0.00 mm, vias 3 -> 0
- net /Pads/I2C0.SCL: track 17.4 -> 0.00 mm, vias 6 -> 0
- net /RX/BOOT: track 16.2 -> 0.00 mm, vias 4 -> 0
- net /RX/SCK: track 16.0 -> 0.00 mm, vias 4 -> 0
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- removed copper zone on F.Cu, net +1.1V
