File: dps/aio/aio.kicad_pcb (KiCad board)
At the start: 8 copper layers, 35 x 35 mm, 280 parts, among them J201 HD VTX, J301 TYPE-C 16P QTWT, J302 TF-021B-H265, J303 GPS (UART3+I2C1), J304 UART4 (MTF-02P), J305 UART1+UART6 (RX, telemetrie), Q10 DOY180N03T, Q11 DOY180N03T, Q12 DOY180N03T, Q13 DOY180N03T, Q14 DOY180N03T, Q15 DOY180N03T, Q16 DOY180N03T, Q17 DOY180N03T, Q18 DOY180N03T, Q19 DOY180N03T, Q20 DOY180N03T, Q21 DOY180N03T, Q22 DOY180N03T, Q23 DOY180N03T, Q24 DOY180N03T, Q25 DOY180N03T, Q26 DOY180N03T, Q3 DOY180N03T, Q301 AP1606, Q4 DOY180N03T, Q5 DOY180N03T, Q6 DOY180N03T, Q7 DOY180N03T, Q8 DOY180N03T, Q9 DOY180N03T, U13 AT32F421G8U7, U14 NSG2065Q, U15 AT32F421G8U7, U16 NSG2065Q, U17 AT32F421G8U7, U18 NSG2065Q, U19 AT32F421G8U7, U20 NSG2065Q, U201 TPS22810DRVR, U24 AIO_outline, U25 INA186A3IDCKR, U3 LMR51430YFDDCR, U301 STM32H743VIH6, U302 SPL06-001 / DPS310, U303 ICM-42688-P, U4 LMR51430YFDDCR, U6 LP5912-1.8DRVR, U7 TLV76733DRVR, U8 BMI270, Y301 8MHz 12pF X32258MOB4SI

Commit message: feat: place each supply capacitor right after its IC, on the nearer side
They used to come after every big part and ended 8-17 mm from U303 and U201;
now they sit 0.7-3.4 mm from their IC.

Co-Authored-By: Claude Opus 5.5 <noreply@anthropic.com>
Parts:
- C201, C202, C203, C318, C319, C324: moved to F.Cu
- moved TP320 25.4 mm to (85.6, 73.0), turned to 0 degrees
- moved R204 24.4 mm to (72.7, 49.3)
- moved R203 23.5 mm to (71.2, 49.6)
- moved C320 22.5 mm to (83.0, 67.6)
- moved C203 22.2 mm to (69.8, 50.8)
- moved C321 20.2 mm to (83.9, 67.8)
- moved R309 18.6 mm to (63.3, 60.7), turned to 90 degrees
- moved TP201 18.3 mm to (85.6, 71.3), turned to 0 degrees
- moved R311 15.9 mm to (76.2, 74.1), turned to 0 degrees
- moved TP322 15.9 mm to (84.9, 53.0), turned to 90 degrees
- moved TP321 14.5 mm to (84.9, 54.3)
- moved C318 13.8 mm to (74.5, 55.8), turned to 0 degrees
- moved R313 12.4 mm to (75.6, 75.7)
- moved TP317 12.4 mm to (87.1, 71.1), turned to 90 degrees
- moved C319 11.7 mm to (76.0, 55.8), turned to 0 degrees
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Routing:
- net GND: vias 856 -> 861
- net /VTX_EN: vias 1 -> 0
- net /MCU H743/UART8_RX: vias 0 -> 2
- net /MCU H743/PWM9: vias 2 -> 0
- net /MCU H743/BOOT0: vias 1 -> 0
- net +3.3V: vias 67 -> 64
